File: Hardware/hydrophone board/hydrophone board.kicad_sch (KiCad schematic)
At the start: 0 parts

Commit message: started layout
Changed lines of the file:
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@@
 (kicad_sch (version 20230121) (generator eeschema)
   (paper "A4")
-  (wire (pts (xy 88.9 76.2) (xy 95.25 76.2))
+  (wire (pts (xy 95.25 88.9) (xy 88.9 88.9))
     (stroke (width 0) (type default))
   )
   (wire (pts (xy 177.8 95.25) (xy 190.5 95.25))
+    (stroke (width 0) (type default))
+  )
+  (wire (pts (xy 114.3 133.35) (xy 127 133.35))
     (stroke (width 0) (type default))
   )
@@
     (stroke (width 0) (type default))
   )
-  (wire (pts (xy 88.9 88.9) (xy 95.25 88.9))
+  (wire (pts (xy 177.8 82.55) (xy 190.5 82.55))
     (stroke (width 0) (type default))
   )
-  (wire (pts (xy 177.8 82.55) (xy 190.5 82.55))
+  (wire (pts (xy 88.9 101.6) (xy 95.25 101.6))
+    (stroke (width 0) (type default))
+  )
+  (wire (pts (xy 146.05 107.95) (xy 146.05 101.6))
+    (stroke (width 0) (type default))
+  )
+  (wire (pts (xy 146.05 57.15) (xy 139.7 57.15))
     (stroke (width 0) (type default))
   )
@@
     (stroke (width 0) (type default))
   )
-  (wire (pts (xy 95.25 101.6) (xy 95.25 107.95))
-    (stroke (width 0) (type default))
-  )
-  (wire (pts (xy 114.3 107.95) (xy 127 107.95))
-    (stroke (width 0) (type default))
-  )
-  (wire (pts (xy 146.05 57.15) (xy 139.7 57.15))
-    (stroke (width 0) (type default))
-  )
-  (wire (pts (xy 146.05 107.95) (xy 146.05 101.6))
-    (stroke (width 0) (type default))
-  )
-  (wire (pts (xy 146.05 101.6) (xy 152.4 101.6))
-    (stroke (width 0) (type default))
-  )
-  (wire (pts (xy 114.3 57.15) (xy 127 57.15))
-    (stroke (width 0) (type default))
-  )
   (wire (pts (xy 146.05 133.35) (xy 146.05 114.3))
     (stroke (width 0) (type default))
   )
-  (wire (pts (xy 114.3 82.55) (xy 127 82.55))
-    (stroke (width 0) (type default))
-  )
   (wire (pts (xy 177.8 114.3) (xy 190.5 114.3))
-    (stroke (width 0) (type default))
-  )
-  (wire (pts (xy 114.3 133.35) (xy 127 133.35))
     (stroke (width 0) (type default))
   )
@@
     (stroke (width 0) (type default))
   )
-  (wire (pts (xy 88.9 101.6) (xy 95.25 101.6))
+  (wire (pts (xy 95.25 57.15) (xy 95.25 76.2))
     (stroke (width 0) (type default))
   )
@@
     (stroke (width 0) (type default))
   )
-  (wire (pts (xy 95.25 57.15) (xy 95.25 76.2))
+  (wire (pts (xy 95.25 101.6) (xy 95.25 107.95))
+    (stroke (width 0) (type default))
+  )
+  (wire (pts (xy 114.3 57.15) (xy 127 57.15))
+    (stroke (width 0) (type default))
+  )
+  (wire (pts (xy 146.05 101.6) (xy 152.4 101.6))
+    (stroke (width 0) (type default))
+  )
+  (wire (pts (xy 114.3 82.55) (xy 127 82.55))
     (stroke (width 0) (type default))
   )
@@
     (stroke (width 0) (type default))
   )
-  (wire (pts (xy 95.25 88.9) (xy 95.25 82.55))
+  (wire (pts (xy 95.25 82.55) (xy 95.25 88.9))
     (stroke (width 0) (type default))
   )
@@
     (stroke (width 0) (type default))
   )
+  (wire (pts (xy 114.3 107.95) (xy 127 107.95))
+    (stroke (width 0) (type default))
+  )
   (wire (pts (xy 177.8 101.6) (xy 190.5 101.6))
+    (stroke (width 0) (type default))
+  )
+  (wire (pts (xy 95.25 76.2) (xy 88.9 76.2))
     (stroke (width 0) (type default))
   )
@@
     (effects (font (size 1.27 1.27)) (justify left bottom))
   )
+  (label "IN_3" (at 95.25 101.6 0) (fields_autoplaced)
+    (effects (font (size 1.27 1.27)) (justify left bottom))
+  )
+  (label "IN_2" (at 95.25 82.55 0) (fields_autoplaced)
+    (effects (font (size 1.27 1.27)) (justify left bottom))
+  )
+  (label "IN_2_B" (at 142.24 82.55 0) (fields_autoplaced)
+    (effects (font (size 1.27 1.27)) (justify left bottom))
+  )
+  (label "IN_4" (at 95.25 133.35 0) (fields_autoplaced)
+    (effects (font (size 1.27 1.27)) (justify left bottom))
+  )
+  (label "IN_1" (at 95.25 57.15 0) (fields_autoplaced)
+    (effects (font (size 1.27 1.27)) (justify left bottom))
+  )
+  (label "IN_4_A" (at 116.84 133.35 0) (fields_autoplaced)
+    (effects (font (size 1.27 1.27)) (justify left bottom))
+  )
+  (label "IN_3_B" (at 142.24 107.95 0) (fields_autoplaced)
+    (effects (font (size 1.27 1.27)) (justify left bottom))
+  )
+  (label "IN_1_B" (at 142.24 57.15 0) (fields_autoplaced)
+    (effects (font (size 1.27 1.27)) (justify left bottom))
+  )
+  (label "IN_1_A" (at 116.84 57.15 0) (fields_autoplaced)
+    (effects (font (size 1.27 1.27)) (justify left bottom))
+  )
+  (label "IN_2_A" (at 116.84 82.55 0) (fields_autoplaced)
+    (effects (font (size 1.27 1.27)) (justify left bottom))
+  )
+  (label "IN_4_B" (at 142.2146 133.35 0) (fields_autoplaced)
+    (effects (font (size 1.27 1.27)) (justify left bottom))
+  )
+  (label "IN_3_A" (at 116.84 107.95 0) (fields_autoplaced)
+    (effects (font (size 1.27 1.27)) (justify left bottom))
+  )
