File: Hardware/hydrophone board/adc.kicad_sch (KiCad schematic)
At the start: 25 parts, among them J301 Conn_01x08

Commit message: adc layout
Parts:
- J301: footprint Connector_PinSocket_2.54mm:PinSocket_1x08_P2.54mm_Vertical -> Connector_PinHeader_2.54mm:PinHeader_1x08_P2.54mm_Vertical
Changed lines of the file:
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@@
       (effects (font (size 1.27 1.27)))
     )
-    (property "Footprint" "Connector_PinSocket_2.54mm:PinSocket_1x08_P2.54mm_Vertical" (at 58.42 99.06 0)
+    (property "Footprint" "Connector_PinHeader_2.54mm:PinHeader_1x08_P2.54mm_Vertical" (at 58.42 99.06 0)
       (effects (font (size 1.27 1.27)) hide)
     )

Commit message: Revert "Merge branch 'hardware' of https://github.com/bruin-underwater-robotics/2023-2024 into hardware"
This reverts commit f5050c74fbd2d727488e15b71bfb24c9149407df, reversing
changes made to d4ffa11f2369dfdbeb25d57bd1642de1ab50c466.
Parts:
- J301: footprint Connector_PinHeader_2.54mm:PinHeader_1x08_P2.54mm_Vertical -> Connector_PinSocket_2.54mm:PinSocket_1x08_P2.54mm_Vertical
Changed lines of the file:
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@@
       (effects (font (size 1.27 1.27)))
     )
-    (property "Footprint" "Connector_PinHeader_2.54mm:PinHeader_1x08_P2.54mm_Vertical" (at 58.42 99.06 0)
+    (property "Footprint" "Connector_PinSocket_2.54mm:PinSocket_1x08_P2.54mm_Vertical" (at 58.42 99.06 0)
       (effects (font (size 1.27 1.27)) hide)
     )
