File: Hardware/hydrophone board/power.kicad_sch (KiCad schematic)
At the start: 17 parts, among them J501 Conn_01x03, U501 LT1963AxST-3.3

Commit message: adc layout
Parts:
- J501: footprint Connector_PinSocket_2.54mm:PinSocket_1x03_P2.54mm_Vertical -> Connector_PinHeader_2.54mm:PinHeader_1x03_P2.54mm_Vertical
Changed lines of the file:
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@@
       (effects (font (size 1.27 1.27)) (justify right))
     )
-    (property "Footprint" "Connector_PinSocket_2.54mm:PinSocket_1x03_P2.54mm_Vertical" (at 143.51 52.07 0)
+    (property "Footprint" "Connector_PinHeader_2.54mm:PinHeader_1x03_P2.54mm_Vertical" (at 143.51 52.07 0)
       (effects (font (size 1.27 1.27)) hide)
     )

Commit message: Revert "Merge branch 'hardware' of https://github.com/bruin-underwater-robotics/2023-2024 into hardware"
This reverts commit f5050c74fbd2d727488e15b71bfb24c9149407df, reversing
changes made to d4ffa11f2369dfdbeb25d57bd1642de1ab50c466.
Parts:
- J501: footprint Connector_PinHeader_2.54mm:PinHeader_1x03_P2.54mm_Vertical -> Connector_PinSocket_2.54mm:PinSocket_1x03_P2.54mm_Vertical
Changed lines of the file:
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@@
       (effects (font (size 1.27 1.27)) (justify right))
     )
-    (property "Footprint" "Connector_PinHeader_2.54mm:PinHeader_1x03_P2.54mm_Vertical" (at 143.51 52.07 0)
+    (property "Footprint" "Connector_PinSocket_2.54mm:PinSocket_1x03_P2.54mm_Vertical" (at 143.51 52.07 0)
       (effects (font (size 1.27 1.27)) hide)
     )
