File: Hardware/hydrophone board/power.kicad_sch (KiCad schematic)
At the start: 17 parts, among them J501 Conn_01x03, U501 LT1963AxST-3.3

Commit message: changed some aprts
Parts:
- removed J501: Conn_01x03, Connector_PinSocket_2.54mm:PinSocket_1x03_P2.54mm_Vertical, symbol Connector_Generic:Conn_01x03
- added JP501: Jumper_3_Bridged12, PCM_4ms_SolderJumper:JUMPER_SMD_1x3, symbol Jumper:Jumper_3_Bridged12
Connections:
- net +3.3VA: now also JP501.2 (C)
- net 3.3V MCU: now also JP501.3 (B)
- net at U501.3 (OUT): now also JP501.1 (A)
Changed lines of the file:
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@@
     (stroke (width 0) (type default))
   )
-  (wire (pts (xy 140.97 76.2) (xy 140.97 57.15))
-    (stroke (width 0) (type default))
-  )
-  (wire (pts (xy 143.51 76.2) (xy 143.51 57.15))
+  (wire (pts (xy 140.97 76.2) (xy 140.97 64.77))
+    (stroke (width 0) (type default))
+  )
+  (wire (pts (xy 143.51 76.2) (xy 143.51 64.77))
+    (stroke (width 0) (type default))
+  )
+  (wire (pts (xy 137.16 64.77) (xy 137.16 60.96))
     (stroke (width 0) (type default))
   )
@@
     (stroke (width 0) (type default))
   )
+  (wire (pts (xy 140.97 64.77) (xy 137.16 64.77))
+    (stroke (width 0) (type default))
+  )
   (wire (pts (xy 107.95 127) (xy 113.03 127))
     (stroke (width 0) (type default))
@@
     (stroke (width 0) (type default))
   )
-  (wire (pts (xy 146.05 57.15) (xy 146.05 60.96))
+  (wire (pts (xy 149.86 60.96) (xy 153.67 60.96))
     (stroke (width 0) (type default))
   )
@@
     (stroke (width 0) (type default))
   )
-  (text "choose 3.3V from MCU or linear regulator" (at 133.35 45.72 0)
+  (text "choose 3.3V from MCU or linear regulator" (at 127 50.8 0)
     (effects (font (size 1.27 1.27)) (justify left bottom))
   )
@@
     (effects (font (size 1.27 1.27)) (justify left bottom))
   )
-  (hierarchical_label "3.3V MCU" (shape input) (at 146.05 60.96 270) (fields_autoplaced)
-    (effects (font (size 1.27 1.27)) (justify right))
+  (hierarchical_label "3.3V MCU" (shape input) (at 153.67 60.96 0) (fields_autoplaced)
+    (effects (font (size 1.27 1.27)) (justify left))
   )
   (symbol (lib_id "Connector:TestPoint_Probe") (at 152.4 76.2 0) (unit 1)
@@
         (path "/4356d3a6-6a00-447d-897e-473f60221539/cf9d259f-9643-49eb-8aca-1ca8b75f4d64"
           (reference "#PWR0506") (unit 1)
-        )
-      )
-    )
-  )
-  (symbol (lib_id "Connector_Generic:Conn_01x03") (at 143.51 52.07 90) (unit 1)
-    (in_bom yes) (on_board yes) (dnp no) (fields_autoplaced)
-    (property "Reference" "J501" (at 148.59 51.435 90)
-      (effects (font (size 1.27 1.27)) (justify right))
-    )
-    (property "Value" "Conn_01x03" (at 148.59 53.975 90)
-      (effects (font (size 1.27 1.27)) (justify right))
-    )
-    (property "Footprint" "Connector_PinSocket_2.54mm:PinSocket_1x03_P2.54mm_Vertical" (at 143.51 52.07 0)
-      (effects (font (size 1.27 1.27)) hide)
-    )
-    (property "Datasheet" "~" (at 143.51 52.07 0)
-      (effects (font (size 1.27 1.27)) hide)
-    )
-    (pin "1")
-    (pin "2")
-    (pin "3")
-    (instances
-      (project "hydrophone board"
-        (path "/4356d3a6-6a00-447d-897e-473f60221539/cf9d259f-9643-49eb-8aca-1ca8b75f4d64"
-          (reference "J501") (unit 1)
         )
       )
@@
         )
       )
+    )
+  )
+  (symbol (lib_id "Jumper:Jumper_3_Bridged12") (at 143.51 60.96 0) (unit 1)
+    (in_bom yes) (on_board yes) (dnp no) (fields_autoplaced)
+    (property "Reference" "JP501" (at 143.51 54.61 0)
+      (effects (font (size 1.27 1.27)))
+    )
+    (property "Value" "Jumper_3_Bridged12" (at 143.51 57.15 0)
+      (effects (font (size 1.27 1.27)))
+    )
+    (property "Footprint" "PCM_4ms_SolderJumper:JUMPER_SMD_1x3" (at 143.51 60.96 0)
+      (effects (font (size 1.27 1.27)) hide)
+    )
+    (property "Datasheet" "~" (at 143.51 60.96 0)
+      (effects (font (size 1.27 1.27)) hide)
+    )
+    (pin "1")
+    (pin "2")
+    (pin "3")
+    (instances
+      (project "hydrophone board"
+        (path "/4356d3a6-6a00-447d-897e-473f60221539/cf9d259f-9643-49eb-8aca-1ca8b75f4d64"
+          (reference "JP501") (unit 1)
+        )
+      )
