File: Hardware/hydrophone board/low pass filter.kicad_sch (KiCad schematic)
At the start: 17 parts, among them U701 AD8648ARZ

Commit message: added teensy footprint
Parts:
- renumbered U701 to U2
Changed lines of the file:
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@@
         )
         (path "/4356d3a6-6a00-447d-897e-473f60221539/c13371a9-09b1-4e65-81c3-6f6fb4c4ebd4"
-          (reference "#PWR0415") (unit 1)
+          (reference "#PWR013") (unit 1)
         )
       )
@@
         )
         (path "/4356d3a6-6a00-447d-897e-473f60221539/c13371a9-09b1-4e65-81c3-6f6fb4c4ebd4"
-          (reference "#PWR0701") (unit 1)
+          (reference "#PWR09") (unit 1)
         )
       )
@@
         )
         (path "/4356d3a6-6a00-447d-897e-473f60221539/c13371a9-09b1-4e65-81c3-6f6fb4c4ebd4"
-          (reference "R411") (unit 1)
+          (reference "R11") (unit 1)
         )
       )
@@
         )
         (path "/4356d3a6-6a00-447d-897e-473f60221539/c13371a9-09b1-4e65-81c3-6f6fb4c4ebd4"
-          (reference "#PWR0704") (unit 1)
+          (reference "#PWR011") (unit 1)
         )
       )
@@
         )
         (path "/4356d3a6-6a00-447d-897e-473f60221539/c13371a9-09b1-4e65-81c3-6f6fb4c4ebd4"
-          (reference "C424") (unit 1)
+          (reference "C11") (unit 1)
         )
       )
@@
   (symbol (lib_id "PCM_Amplifier_Operational_AKL:AD8648ARZ") (at 177.8 82.55 0) (unit 3)
     (in_bom yes) (on_board yes) (dnp no) (fields_autoplaced)
-    (property "Reference" "U701" (at 179.07 73.66 0)
+    (property "Reference" "U2" (at 179.07 73.66 0)
       (effects (font (size 1.27 1.27)))
     )
@@
       (project "hydrophone board"
         (path "/4356d3a6-6a00-447d-897e-473f60221539/c13371a9-09b1-4e65-81c3-6f6fb4c4ebd4"
-          (reference "U701") (unit 3)
+          (reference "U2") (unit 3)
         )
       )
@@
         )
         (path "/4356d3a6-6a00-447d-897e-473f60221539/c13371a9-09b1-4e65-81c3-6f6fb4c4ebd4"
-          (reference "R406") (unit 1)
+          (reference "R6") (unit 1)
         )
       )
@@
         )
         (path "/4356d3a6-6a00-447d-897e-473f60221539/c13371a9-09b1-4e65-81c3-6f6fb4c4ebd4"
-          (reference "TP409") (unit 1)
+          (reference "TP2") (unit 1)
         )
       )
@@
         )
         (path "/4356d3a6-6a00-447d-897e-473f60221539/c13371a9-09b1-4e65-81c3-6f6fb4c4ebd4"
-          (reference "R407") (unit 1)
+          (reference "R7") (unit 1)
         )
       )
@@
         )
         (path "/4356d3a6-6a00-447d-897e-473f60221539/c13371a9-09b1-4e65-81c3-6f6fb4c4ebd4"
-          (reference "C425") (unit 1)
+          (reference "C12") (unit 1)
         )
       )
@@
   (symbol (lib_id "PCM_Amplifier_Operational_AKL:AD8648ARZ") (at 76.2 87.63 0) (unit 1)
     (in_bom yes) (on_board yes) (dnp no) (fields_autoplaced)
-    (property "Reference" "U701" (at 88.9 84.2011 0)
+    (property "Reference" "U2" (at 88.9 84.2011 0)
       (effects (font (size 1.27 1.27)))
     )
@@
       (project "hydrophone board"
         (path "/4356d3a6-6a00-447d-897e-473f60221539/c13371a9-09b1-4e65-81c3-6f6fb4c4ebd4"
-          (reference "U701") (unit 1)
+          (reference "U2") (unit 1)
         )
       )
@@
         )
         (path "/4356d3a6-6a00-447d-897e-473f60221539/c13371a9-09b1-4e65-81c3-6f6fb4c4ebd4"
-          (reference "R409") (unit 1)
+          (reference "R9") (unit 1)
         )
       )
@@
         )
         (path "/4356d3a6-6a00-447d-897e-473f60221539/c13371a9-09b1-4e65-81c3-6f6fb4c4ebd4"
-          (reference "#PWR0417") (unit 1)
+          (reference "#PWR015") (unit 1)
         )
       )
@@
         )
         (path "/4356d3a6-6a00-447d-897e-473f60221539/c13371a9-09b1-4e65-81c3-6f6fb4c4ebd4"
-          (reference "C703") (unit 1)
+          (reference "C6") (unit 1)
         )
       )
@@
         )
         (path "/4356d3a6-6a00-447d-897e-473f60221539/c13371a9-09b1-4e65-81c3-6f6fb4c4ebd4"
-          (reference "R408") (unit 1)
+          (reference "R8") (unit 1)
         )
       )
@@
         )
         (path "/4356d3a6-6a00-447d-897e-473f60221539/c13371a9-09b1-4e65-81c3-6f6fb4c4ebd4"
-          (reference "C701") (unit 1)
+          (reference "C5") (unit 1)
         )
       )
@@
   (symbol (lib_id "PCM_Amplifier_Operational_AKL:AD8648ARZ") (at 127 85.09 0) (unit 2)
     (in_bom yes) (on_board yes) (dnp no) (fields_autoplaced)
-    (property "Reference" "U701" (at 128.27 76.2 0)
+    (property "Reference" "U2" (at 128.27 76.2 0)
       (effects (font (size 1.27 1.27)))
     )
@@
       (project "hydrophone board"
         (path "/4356d3a6-6a00-447d-897e-473f60221539/c13371a9-09b1-4e65-81c3-6f6fb4c4ebd4"
-          (reference "U701") (unit 2)
+          (reference "U2") (unit 2)
         )
       )
@@
         )
         (path "/4356d3a6-6a00-447d-897e-473f60221539/c13371a9-09b1-4e65-81c3-6f6fb4c4ebd4"
-          (reference "R702") (unit 1)
+          (reference "R5") (unit 1)
         )
       )
@@
         )
         (path "/4356d3a6-6a00-447d-897e-473f60221539/c13371a9-09b1-4e65-81c3-6f6fb4c4ebd4"
-          (reference "R410") (unit 1)
+          (reference "R10") (unit 1)
         )
       )
@@
         )
         (path "/4356d3a6-6a00-447d-897e-473f60221539/c13371a9-09b1-4e65-81c3-6f6fb4c4ebd4"
-          (reference "#PWR0702") (unit 1)
+          (reference "#PWR010") (unit 1)
         )
       )
@@
         )
         (path "/4356d3a6-6a00-447d-897e-473f60221539/c13371a9-09b1-4e65-81c3-6f6fb4c4ebd4"
-          (reference "C420") (unit 1)
+          (reference "C8") (unit 1)
         )
       )
@@
         )
         (path "/4356d3a6-6a00-447d-897e-473f60221539/c13371a9-09b1-4e65-81c3-6f6fb4c4ebd4"
-          (reference "C421") (unit 1)
+          (reference "C7") (unit 1)
         )
       )
@@
         )
         (path "/4356d3a6-6a00-447d-897e-473f60221539/c13371a9-09b1-4e65-81c3-6f6fb4c4ebd4"
-          (reference "#PWR0416") (unit 1)
+          (reference "#PWR014") (unit 1)
         )
       )
@@
         )
         (path "/4356d3a6-6a00-447d-897e-473f60221539/c13371a9-09b1-4e65-81c3-6f6fb4c4ebd4"
-          (reference "#PWR0703") (unit 1)
+          (reference "#PWR012") (unit 1)
         )
       )
@@
         )
         (path "/4356d3a6-6a00-447d-897e-473f60221539/c13371a9-09b1-4e65-81c3-6f6fb4c4ebd4"
-          (reference "C422") (unit 1)
+          (reference "C9") (unit 1)
         )
       )
@@
         )
         (path "/4356d3a6-6a00-447d-897e-473f60221539/c13371a9-09b1-4e65-81c3-6f6fb4c4ebd4"
-          (reference "C423") (unit 1)
+          (reference "C10") (unit 1)
         )
       )
@@
   (symbol (lib_id "PCM_Amplifier_Operational_AKL:AD8648ARZ") (at 228.6 80.01 0) (unit 4)
     (in_bom yes) (on_board yes) (dnp no) (fields_autoplaced)
-    (property "Reference" "U701" (at 229.87 71.12 0)
+    (property "Reference" "U2" (at 229.87 71.12 0)
       (effects (font (size 1.27 1.27)))
     )
@@
       (project "hydrophone board"
         (path "/4356d3a6-6a00-447d-897e-473f60221539/c13371a9-09b1-4e65-81c3-6f6fb4c4ebd4"
-          (reference "U701") (unit 4)
-        )
-      )
+          (reference "U2") (unit 4)
+        )
+      )

Commit message: annotate all component
Parts:
- renumbered U2 to U211

Commit message: assigned footprints
Parts:
- C303, C304, C305: footprint (none) -> Capacitor_SMD:C_0603_1608Metric
- R306, R307: footprint (none) -> Resistor_SMD:R_0603_1608Metric
- TP?: footprint (none) -> Connector_PinHeader_2.54mm:PinHeader_1x01_P2.54mm_Vertical
Changed lines of the file:
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@@
       (effects (font (size 1.27 1.27)))
     )
-    (property "Footprint" "" (at 209.804 81.534 90)
+    (property "Footprint" "Resistor_SMD:R_0603_1608Metric" (at 209.804 81.534 90)
       (effects (font (size 1.27 1.27)) hide)
     )
@@
       (effects (font (size 1.27 1.27)) (justify right))
     )
-    (property "Footprint" "" (at 214.9348 87.63 0)
+    (property "Footprint" "Capacitor_SMD:C_0603_1608Metric" (at 214.9348 87.63 0)
       (effects (font (size 1.27 1.27)) hide)
     )
@@
       (effects (font (size 1.27 1.27)))
     )
-    (property "Footprint" "" (at 95.504 86.614 90)
+    (property "Footprint" "Resistor_SMD:R_0603_1608Metric" (at 95.504 86.614 90)
       (effects (font (size 1.27 1.27)) hide)
     )
@@
       (effects (font (size 1.27 1.27)) (justify left))
     )
-    (property "Footprint" "" (at 252.73 73.66 0)
+    (property "Footprint" "Connector_PinHeader_2.54mm:PinHeader_1x01_P2.54mm_Vertical" (at 252.73 73.66 0)
       (effects (font (size 1.27 1.27)) hide)
     )
@@
       (effects (font (size 1.27 1.27)))
     )
-    (property "Footprint" "" (at 108.204 86.614 90)
+    (property "Footprint" "Resistor_SMD:R_0603_1608Metric" (at 108.204 86.614 90)
       (effects (font (size 1.27 1.27)) hide)
     )
@@
       (effects (font (size 1.27 1.27)))
     )
-    (property "Footprint" "" (at 218.44 67.0052 0)
+    (property "Footprint" "Capacitor_SMD:C_0603_1608Metric" (at 218.44 67.0052 0)
       (effects (font (size 1.27 1.27)) hide)
     )
@@
       (effects (font (size 1.27 1.27)))
     )
-    (property "Footprint" "" (at 159.004 84.074 90)
+    (property "Footprint" "Resistor_SMD:R_0603_1608Metric" (at 159.004 84.074 90)
       (effects (font (size 1.27 1.27)) hide)
     )
@@
       (effects (font (size 1.27 1.27)))
     )
-    (property "Footprint" "" (at 87.63 68.8848 0)
+    (property "Footprint" "Capacitor_SMD:C_0603_1608Metric" (at 87.63 68.8848 0)
       (effects (font (size 1.27 1.27)) hide)
     )
@@
       (effects (font (size 1.27 1.27)))
     )
-    (property "Footprint" "" (at 146.304 84.074 90)
+    (property "Footprint" "Resistor_SMD:R_0603_1608Metric" (at 146.304 84.074 90)
       (effects (font (size 1.27 1.27)) hide)
     )
@@
       (effects (font (size 1.27 1.27)) (justify right))
     )
-    (property "Footprint" "" (at 62.5348 95.25 0)
+    (property "Footprint" "Capacitor_SMD:C_0603_1608Metric" (at 62.5348 95.25 0)
       (effects (font (size 1.27 1.27)) hide)
     )
@@
       (effects (font (size 1.27 1.27)))
     )
-    (property "Footprint" "" (at 57.404 89.154 90)
+    (property "Footprint" "Resistor_SMD:R_0603_1608Metric" (at 57.404 89.154 90)
       (effects (font (size 1.27 1.27)) hide)
     )
@@
       (effects (font (size 1.27 1.27)))
     )
-    (property "Footprint" "" (at 197.104 81.534 90)
+    (property "Footprint" "Resistor_SMD:R_0603_1608Metric" (at 197.104 81.534 90)
       (effects (font (size 1.27 1.27)) hide)
     )
@@
       (effects (font (size 1.27 1.27)))
     )
-    (property "Footprint" "" (at 116.84 72.0852 0)
+    (property "Footprint" "Capacitor_SMD:C_0603_1608Metric" (at 116.84 72.0852 0)
       (effects (font (size 1.27 1.27)) hide)
     )
@@
       (effects (font (size 1.27 1.27)) (justify right))
     )
-    (property "Footprint" "" (at 113.3348 92.71 0)
+    (property "Footprint" "Capacitor_SMD:C_0603_1608Metric" (at 113.3348 92.71 0)
       (effects (font (size 1.27 1.27)) hide)
     )
@@
       (effects (font (size 1.27 1.27)) (justify right))
     )
-    (property "Footprint" "" (at 164.1348 90.17 0)
+    (property "Footprint" "Capacitor_SMD:C_0603_1608Metric" (at 164.1348 90.17 0)
       (effects (font (size 1.27 1.27)) hide)
     )
@@
       (effects (font (size 1.27 1.27)))
     )
-    (property "Footprint" "" (at 167.64 69.5452 0)
-      (effects (font (size 1.27 1.27)) hide)
-    )
+    (property "Footprint" "Capacitor_SMD:C_0603_1608Metric" (at 167.64 69.5452 0)
+      (effects (font (size 1.27 1.27)) hide)
+    )

Commit message: changed low pass filter op amp
Parts:
- removed U211: AD8648ARZ, Package_SO_AKL:SOIC-14_3.9x8.7mm_P1.27mm, symbol PCM_Amplifier_Operational_AKL:AD8648ARZ
- added U211: AD8544ARZ, Package_SO_AKL:SOIC-14_3.9x8.7mm_P1.27mm, symbol PCM_Amplifier_Operational_AKL:AD8544ARZ
Connections:
- net +3.3VA: now also U211.4 (V+)
- net GND: now also U211.11 (V-)
- net OUT: now also U211.13 (-), U211.14
- net at C304.2, R306.2: now also U211.12 (+)
- net at C304.2, R306.2: now also U211.10 (+)
- net at C305.1, R306.1: now also U211.8, U211.9 (-)
- net at R306.1: now also U211.1, U211.2 (-)
- net at C304.2, R306.2: now also U211.5 (+)
- net at C304.2, R307.2: now also U211.3 (+)
- net at C305.1, R306.1: now also U211.6 (-), U211.7

Commit message: unchanged low pass filter op amp
Parts:
- removed U211: AD8544ARZ, Package_SO_AKL:SOIC-14_3.9x8.7mm_P1.27mm, symbol PCM_Amplifier_Operational_AKL:AD8544ARZ
- added U211: AD8648ARZ, Package_SO_AKL:SOIC-14_3.9x8.7mm_P1.27mm, symbol PCM_Amplifier_Operational_AKL:AD8648ARZ
Connections:
- net +3.3VA: now also U211.4 (V+)
- net GND: now also U211.11 (V-)
- net OUT: now also U211.13 (-), U211.14
- net at C304.2, R306.2: now also U211.12 (+)
- net at C304.2, R306.2: now also U211.10 (+)
- net at C305.1, R306.1: now also U211.8, U211.9 (-)
- net at R306.1: now also U211.1, U211.2 (-)
- net at C304.2, R307.2: now also U211.3 (+)
- net at C304.2, R306.2: now also U211.5 (+)
- net at C305.1, R306.1: now also U211.6 (-), U211.7

Commit message: changed all cap + resistors to 0805, starting filter layout
Parts:
- C303, C304, C305: footprint Capacitor_SMD:C_0603_1608Metric -> Capacitor_SMD:C_0805_2012Metric_Pad1.18x1.45mm_HandSolder
- R306, R307: footprint Resistor_SMD:R_0603_1608Metric -> Resistor_SMD:R_0805_2012Metric_Pad1.20x1.40mm_HandSolder
Changed lines of the file:
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@@
       (effects (font (size 1.27 1.27)))
     )
-    (property "Footprint" "Resistor_SMD:R_0603_1608Metric" (at 209.804 81.534 90)
+    (property "Footprint" "Resistor_SMD:R_0805_2012Metric_Pad1.20x1.40mm_HandSolder" (at 209.804 81.534 90)
       (effects (font (size 1.27 1.27)) hide)
     )
@@
       (effects (font (size 1.27 1.27)) (justify right))
     )
-    (property "Footprint" "Capacitor_SMD:C_0603_1608Metric" (at 214.9348 87.63 0)
+    (property "Footprint" "Capacitor_SMD:C_0805_2012Metric_Pad1.18x1.45mm_HandSolder" (at 214.9348 87.63 0)
       (effects (font (size 1.27 1.27)) hide)
     )
@@
       (effects (font (size 1.27 1.27)))
     )
-    (property "Footprint" "Resistor_SMD:R_0603_1608Metric" (at 95.504 86.614 90)
+    (property "Footprint" "Resistor_SMD:R_0805_2012Metric_Pad1.20x1.40mm_HandSolder" (at 95.504 86.614 90)
       (effects (font (size 1.27 1.27)) hide)
     )
@@
       (effects (font (size 1.27 1.27)))
     )
-    (property "Footprint" "Resistor_SMD:R_0603_1608Metric" (at 108.204 86.614 90)
+    (property "Footprint" "Resistor_SMD:R_0805_2012Metric_Pad1.20x1.40mm_HandSolder" (at 108.204 86.614 90)
       (effects (font (size 1.27 1.27)) hide)
     )
@@
       (effects (font (size 1.27 1.27)))
     )
-    (property "Footprint" "Capacitor_SMD:C_0603_1608Metric" (at 218.44 67.0052 0)
+    (property "Footprint" "Capacitor_SMD:C_0805_2012Metric_Pad1.18x1.45mm_HandSolder" (at 218.44 67.0052 0)
       (effects (font (size 1.27 1.27)) hide)
     )
@@
       (effects (font (size 1.27 1.27)))
     )
-    (property "Footprint" "Resistor_SMD:R_0603_1608Metric" (at 159.004 84.074 90)
+    (property "Footprint" "Resistor_SMD:R_0805_2012Metric_Pad1.20x1.40mm_HandSolder" (at 159.004 84.074 90)
       (effects (font (size 1.27 1.27)) hide)
     )
@@
       (effects (font (size 1.27 1.27)))
     )
-    (property "Footprint" "Capacitor_SMD:C_0603_1608Metric" (at 87.63 68.8848 0)
+    (property "Footprint" "Capacitor_SMD:C_0805_2012Metric_Pad1.18x1.45mm_HandSolder" (at 87.63 68.8848 0)
       (effects (font (size 1.27 1.27)) hide)
     )
@@
       (effects (font (size 1.27 1.27)))
     )
-    (property "Footprint" "Resistor_SMD:R_0603_1608Metric" (at 146.304 84.074 90)
+    (property "Footprint" "Resistor_SMD:R_0805_2012Metric_Pad1.20x1.40mm_HandSolder" (at 146.304 84.074 90)
       (effects (font (size 1.27 1.27)) hide)
     )
@@
       (effects (font (size 1.27 1.27)) (justify right))
     )
-    (property "Footprint" "Capacitor_SMD:C_0603_1608Metric" (at 62.5348 95.25 0)
+    (property "Footprint" "Capacitor_SMD:C_0805_2012Metric_Pad1.18x1.45mm_HandSolder" (at 62.5348 95.25 0)
       (effects (font (size 1.27 1.27)) hide)
     )
@@
       (effects (font (size 1.27 1.27)))
     )
-    (property "Footprint" "Resistor_SMD:R_0603_1608Metric" (at 57.404 89.154 90)
+    (property "Footprint" "Resistor_SMD:R_0805_2012Metric_Pad1.20x1.40mm_HandSolder" (at 57.404 89.154 90)
       (effects (font (size 1.27 1.27)) hide)
     )
@@
       (effects (font (size 1.27 1.27)))
     )
-    (property "Footprint" "Resistor_SMD:R_0603_1608Metric" (at 197.104 81.534 90)
+    (property "Footprint" "Resistor_SMD:R_0805_2012Metric_Pad1.20x1.40mm_HandSolder" (at 197.104 81.534 90)
       (effects (font (size 1.27 1.27)) hide)
     )
@@
       (effects (font (size 1.27 1.27)))
     )
-    (property "Footprint" "Capacitor_SMD:C_0603_1608Metric" (at 116.84 72.0852 0)
+    (property "Footprint" "Capacitor_SMD:C_0805_2012Metric_Pad1.18x1.45mm_HandSolder" (at 116.84 72.0852 0)
       (effects (font (size 1.27 1.27)) hide)
     )
@@
       (effects (font (size 1.27 1.27)) (justify right))
     )
-    (property "Footprint" "Capacitor_SMD:C_0603_1608Metric" (at 113.3348 92.71 0)
+    (property "Footprint" "Capacitor_SMD:C_0805_2012Metric_Pad1.18x1.45mm_HandSolder" (at 113.3348 92.71 0)
       (effects (font (size 1.27 1.27)) hide)
     )
@@
       (effects (font (size 1.27 1.27)) (justify right))
     )
-    (property "Footprint" "Capacitor_SMD:C_0603_1608Metric" (at 164.1348 90.17 0)
+    (property "Footprint" "Capacitor_SMD:C_0805_2012Metric_Pad1.18x1.45mm_HandSolder" (at 164.1348 90.17 0)
       (effects (font (size 1.27 1.27)) hide)
     )
@@
       (effects (font (size 1.27 1.27)))
     )
-    (property "Footprint" "Capacitor_SMD:C_0603_1608Metric" (at 167.64 69.5452 0)
-      (effects (font (size 1.27 1.27)) hide)
-    )
+    (property "Footprint" "Capacitor_SMD:C_0805_2012Metric_Pad1.18x1.45mm_HandSolder" (at 167.64 69.5452 0)
+      (effects (font (size 1.27 1.27)) hide)
+    )
