File: Hardware/hydrophone board/low pass filter.kicad_sch (KiCad schematic)
At the start: 17 parts, among them U211 AD8648ARZ

Commit message: changed some aprts
Parts:
- removed TP?: TestPoint_Probe, Connector_PinHeader_2.54mm:PinHeader_1x01_P2.54mm_Vertical, symbol Connector:TestPoint_Probe
- added J5: Conn_01x02, Connector_PinHeader_2.54mm:PinHeader_1x02_P2.54mm_Vertical, symbol Connector_Generic:Conn_01x02
Connections:
- net GND: now also J5.1 (Pin_1)
- net OUT: now also J5.2 (Pin_2)
Changed lines of the file:
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@@
 (kicad_sch (version 20230121) (generator eeschema)
   (paper "A4")
-  (junction (at 247.65 80.01) (diameter 0) (color 0 0 0 0)
-  )
   (junction (at 139.7 85.09) (diameter 0) (color 0 0 0 0)
   )
@@
     (stroke (width 0) (type default))
   )
+  (wire (pts (xy 241.3 92.71) (xy 241.3 97.79))
+    (stroke (width 0) (type default))
+  )
   (wire (pts (xy 85.09 87.63) (xy 88.9 87.63))
     (stroke (width 0) (type default))
   )
+  (wire (pts (xy 241.3 80.01) (xy 254 80.01))
+    (stroke (width 0) (type default))
+  )
   (wire (pts (xy 200.66 82.55) (xy 203.2 82.55))
     (stroke (width 0) (type default))
@@
     (stroke (width 0) (type default))
   )
-  (wire (pts (xy 247.65 73.66) (xy 247.65 80.01))
-    (stroke (width 0) (type default))
-  )
   (wire (pts (xy 203.2 82.55) (xy 205.74 82.55))
     (stroke (width 0) (type default))
@@
     (stroke (width 0) (type default))
   )
-  (wire (pts (xy 241.3 80.01) (xy 247.65 80.01))
-    (stroke (width 0) (type default))
-  )
   (wire (pts (xy 139.7 77.47) (xy 139.7 85.09))
     (stroke (width 0) (type default))
@@
     (stroke (width 0) (type default))
   )
-  (wire (pts (xy 247.65 80.01) (xy 254 80.01))
+  (wire (pts (xy 241.3 80.01) (xy 241.3 90.17))
     (stroke (width 0) (type default))
   )
@@
   (hierarchical_label "OUT" (shape output) (at 254 80.01 0) (fields_autoplaced)
     (effects (font (size 1.27 1.27)) (justify left))
+  )
+  (symbol (lib_id "power:GND") (at 241.3 97.79 0) (unit 1)
+    (in_bom yes) (on_board yes) (dnp no) (fields_autoplaced)
+    (property "Reference" "#PWR0205" (at 241.3 104.14 0)
+      (effects (font (size 1.27 1.27)) hide)
+    )
+    (property "Value" "GND" (at 241.3 102.87 0)
+      (effects (font (size 1.27 1.27)))
+    )
+    (property "Footprint" "" (at 241.3 97.79 0)
+      (effects (font (size 1.27 1.27)) hide)
+    )
+    (property "Datasheet" "" (at 241.3 97.79 0)
+      (effects (font (size 1.27 1.27)) hide)
+    )
+    (pin "1")
+    (instances
+      (project "hydrophone board"
+        (path "/4356d3a6-6a00-447d-897e-473f60221539/1cfbaf71-7039-4355-8fc7-d8c77f0e8058"
+          (reference "#PWR0205") (unit 1)
+        )
+        (path "/4356d3a6-6a00-447d-897e-473f60221539/f560d530-135c-40dc-9144-4f9599a30f13"
+          (reference "#PWR0252") (unit 1)
+        )
+        (path "/4356d3a6-6a00-447d-897e-473f60221539/fa1a46a1-ed86-4a84-a182-b5dbe7fc86e7"
+          (reference "#PWR0253") (unit 1)
+        )
+        (path "/4356d3a6-6a00-447d-897e-473f60221539/d3a562a3-af99-4bb5-b5fa-eb83660cffa4"
+          (reference "#PWR0254") (unit 1)
+        )
+        (path "/4356d3a6-6a00-447d-897e-473f60221539/6f981a72-1f6f-4ccf-ba7d-c5dfb70b4229"
+          (reference "#PWR0255") (unit 1)
+        )
+        (path "/4356d3a6-6a00-447d-897e-473f60221539/c13371a9-09b1-4e65-81c3-6f6fb4c4ebd4"
+          (reference "#PWR0256") (unit 1)
+        )
+        (path "/4356d3a6-6a00-447d-897e-473f60221539/924dcbbe-1ff5-4b2e-a973-2a9e51c40258"
+          (reference "#PWR0257") (unit 1)
+        )
+        (path "/4356d3a6-6a00-447d-897e-473f60221539/9c7eb115-b279-4a21-9abb-ee1a14da0145"
+          (reference "#PWR0258") (unit 1)
+        )
+        (path "/4356d3a6-6a00-447d-897e-473f60221539/025ca7c2-0364-4e32-8d6c-dbe542d6c74c"
+          (reference "#PWR0259") (unit 1)
+        )
+      )
+    )
   )
   (symbol (lib_id "power:GND") (at 114.3 105.41 0) (unit 1)
@@
     )
   )
-  (symbol (lib_id "Connector:TestPoint_Probe") (at 247.65 73.66 0) (unit 1)
-    (in_bom yes) (on_board yes) (dnp no) (fields_autoplaced)
-    (property "Reference" "TP?" (at 251.46 71.4375 0)
-      (effects (font (size 1.27 1.27)) (justify left))
-    )
-    (property "Value" "TestPoint_Probe" (at 251.46 73.9775 0)
-      (effects (font (size 1.27 1.27)) (justify left))
-    )
-    (property "Footprint" "Connector_PinHeader_2.54mm:PinHeader_1x01_P2.54mm_Vertical" (at 252.73 73.66 0)
-      (effects (font (size 1.27 1.27)) hide)
-    )
-    (property "Datasheet" "~" (at 252.73 73.66 0)
-      (effects (font (size 1.27 1.27)) hide)
-    )
-    (pin "1")
-    (instances
-      (project "hydrophone board"
-        (path "/4356d3a6-6a00-447d-897e-473f60221539/cf9d259f-9643-49eb-8aca-1ca8b75f4d64"
-          (reference "TP?") (unit 1)
-        )
-        (path "/4356d3a6-6a00-447d-897e-473f60221539/f560d530-135c-40dc-9144-4f9599a30f13"
-          (reference "TP301") (unit 1)
-        )
-        (path "/4356d3a6-6a00-447d-897e-473f60221539/c13371a9-09b1-4e65-81c3-6f6fb4c4ebd4"
-          (reference "TP211") (unit 1)
-        )
-        (path "/4356d3a6-6a00-447d-897e-473f60221539/924dcbbe-1ff5-4b2e-a973-2a9e51c40258"
-          (reference "TP221") (unit 1)
-        )
-        (path "/4356d3a6-6a00-447d-897e-473f60221539/9c7eb115-b279-4a21-9abb-ee1a14da0145"
-          (reference "TP231") (unit 1)
-        )
-        (path "/4356d3a6-6a00-447d-897e-473f60221539/025ca7c2-0364-4e32-8d6c-dbe542d6c74c"
-          (reference "TP241") (unit 1)
-        )
-      )
-    )
-  )
   (symbol (lib_id "Device:R_US") (at 107.95 87.63 90) (unit 1)
     (in_bom yes) (on_board yes) (dnp no) (fields_autoplaced)
@@
         )
       )
+    )
+  )
+  (symbol (lib_id "Connector_Generic:Conn_01x02") (at 236.22 92.71 180) (unit 1)
+    (in_bom yes) (on_board yes) (dnp no)
+    (property "Reference" "J5" (at 236.22 83.82 0)
+      (effects (font (size 1.27 1.27)))
+    )
+    (property "Value" "Conn_01x02" (at 236.22 86.36 0)
+      (effects (font (size 1.27 1.27)))
+    )
+    (property "Footprint" "Connector_PinHeader_2.54mm:PinHeader_1x02_P2.54mm_Vertical" (at 236.22 92.71 0)
+      (effects (font (size 1.27 1.27)) hide)
+    )
+    (property "Datasheet" "~" (at 236.22 92.71 0)
+      (effects (font (size 1.27 1.27)) hide)
+    )
+    (pin "1")
+    (pin "2")
+    (instances
+      (project "hydrophone board"
+        (path "/4356d3a6-6a00-447d-897e-473f60221539/1cfbaf71-7039-4355-8fc7-d8c77f0e8058"
+          (reference "J5") (unit 1)
+        )
+        (path "/4356d3a6-6a00-447d-897e-473f60221539/f560d530-135c-40dc-9144-4f9599a30f13"
+          (reference "J111") (unit 1)
+        )
+        (path "/4356d3a6-6a00-447d-897e-473f60221539/fa1a46a1-ed86-4a84-a182-b5dbe7fc86e7"
+          (reference "J242") (unit 1)
+        )
+        (path "/4356d3a6-6a00-447d-897e-473f60221539/d3a562a3-af99-4bb5-b5fa-eb83660cffa4"
+          (reference "J243") (unit 1)
+        )
+        (path "/4356d3a6-6a00-447d-897e-473f60221539/6f981a72-1f6f-4ccf-ba7d-c5dfb70b4229"
+          (reference "J244") (unit 1)
+        )
+        (path "/4356d3a6-6a00-447d-897e-473f60221539/c13371a9-09b1-4e65-81c3-6f6fb4c4ebd4"
+          (reference "J211") (unit 1)
+        )
+        (path "/4356d3a6-6a00-447d-897e-473f60221539/924dcbbe-1ff5-4b2e-a973-2a9e51c40258"
+          (reference "J221") (unit 1)
+        )
+        (path "/4356d3a6-6a00-447d-897e-473f60221539/9c7eb115-b279-4a21-9abb-ee1a14da0145"
+          (reference "J231") (unit 1)
+        )
+        (path "/4356d3a6-6a00-447d-897e-473f60221539/025ca7c2-0364-4e32-8d6c-dbe542d6c74c"
+          (reference "J241") (unit 1)
+        )
+      )
