File: Hardware/battery monitoring board/e-switch_sch.kicad_sch (KiCad schematic)
At the start: 0 parts

Commit message: Update e-switch_sch.kicad_sch
Parts:
- added D1: D_Zener, symbol Device:D_Zener
- added Q1: PMOS, symbol Simulation_SPICE:PMOS
- added Q2: NMOS, symbol Simulation_SPICE:NMOS
- added R1, R2, R3, R4: R_US, symbol Device:R_US
Connections:
- new net: D1.2 (A), Q1.2 (G), R1.2, R2.1
- new net: Q2.1 (D), R2.2
- new net: D1.1 (K), Q1.1 (D), R1.1
- new net: Q2.2 (G), R3.2, R4.1
- new net GND: Q2.3 (S), R4.2
- new net MCU: R3.1

Commit message: leak sensor schema
Parts:
- removed D1: D_Zener, symbol Device:D_Zener
- removed Q1: PMOS, symbol Simulation_SPICE:PMOS
- removed Q2: NMOS, symbol Simulation_SPICE:NMOS
- removed R1, R2, R3, R4: R_US, symbol Device:R_US
