File: Hardware/battery monitoring board/e-switch_sch.kicad_sch (KiCad schematic)
At the start: 10 parts, among them J5 - 9V BAT +, K1 Relay_SPST-NO, Q2 PN2222A

Commit message: finalized battery board !!
Parts:
- renumbered D7 to D6, R17 to R16, R19 to R18
Changed lines of the file:
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@@
         )
         (path "/bf623d80-ca5a-491f-9daa-4dffbeba5279/d1e89632-1041-42ed-815d-03472eda859a"
-          (reference "TP14") (unit 1)
+          (reference "TP2") (unit 1)
         )
       )
@@
   (symbol (lib_id "power:GND") (at 86.36 92.71 0) (unit 1)
     (in_bom yes) (on_board yes) (dnp no) (fields_autoplaced)
-    (property "Reference" "#PWR031" (at 86.36 99.06 0)
+    (property "Reference" "#PWR032" (at 86.36 99.06 0)
       (effects (font (size 1.27 1.27)) hide)
     )
@@
       (project "battery monitoring board"
         (path "/bf623d80-ca5a-491f-9daa-4dffbeba5279/d1e89632-1041-42ed-815d-03472eda859a"
-          (reference "#PWR031") (unit 1)
+          (reference "#PWR032") (unit 1)
         )
       )
@@
         )
         (path "/bf623d80-ca5a-491f-9daa-4dffbeba5279/d1e89632-1041-42ed-815d-03472eda859a"
-          (reference "R18") (unit 1)
+          (reference "R17") (unit 1)
         )
       )
@@
         )
         (path "/bf623d80-ca5a-491f-9daa-4dffbeba5279/d1e89632-1041-42ed-815d-03472eda859a"
-          (reference "J9") (unit 1)
+          (reference "J10") (unit 1)
         )
       )
@@
   (symbol (lib_id "PCM_4ms_Power-symbol:GND") (at 44.45 50.8 0) (unit 1)
     (in_bom yes) (on_board yes) (dnp no) (fields_autoplaced)
-    (property "Reference" "#PWR030" (at 44.45 57.15 0)
+    (property "Reference" "#PWR031" (at 44.45 57.15 0)
       (effects (font (size 1.27 1.27)) hide)
     )
@@
       (project "battery monitoring board"
         (path "/bf623d80-ca5a-491f-9daa-4dffbeba5279/d1e89632-1041-42ed-815d-03472eda859a"
+          (reference "#PWR031") (unit 1)
+        )
+      )
+    )
+  )
+  (symbol (lib_id "PCM_4ms_Power-symbol:+9V") (at 44.45 44.45 0) (unit 1)
+    (in_bom yes) (on_board yes) (dnp no) (fields_autoplaced)
+    (property "Reference" "#PWR030" (at 44.45 48.26 0)
+      (effects (font (size 1.27 1.27)) hide)
+    )
+    (property "Value" "+9V" (at 44.45 39.37 0)
+      (effects (font (size 1.27 1.27)))
+    )
+    (property "Footprint" "" (at 44.45 44.45 0)
+      (effects (font (size 1.27 1.27)) hide)
+    )
+    (property "Datasheet" "" (at 44.45 44.45 0)
+      (effects (font (size 1.27 1.27)) hide)
+    )
+    (pin "1")
+    (instances
+      (project "battery monitoring board"
+        (path "/bf623d80-ca5a-491f-9daa-4dffbeba5279/d1e89632-1041-42ed-815d-03472eda859a"
           (reference "#PWR030") (unit 1)
-        )
-      )
-    )
-  )
-  (symbol (lib_id "PCM_4ms_Power-symbol:+9V") (at 44.45 44.45 0) (unit 1)
-    (in_bom yes) (on_board yes) (dnp no) (fields_autoplaced)
-    (property "Reference" "#PWR029" (at 44.45 48.26 0)
-      (effects (font (size 1.27 1.27)) hide)
-    )
-    (property "Value" "+9V" (at 44.45 39.37 0)
-      (effects (font (size 1.27 1.27)))
-    )
-    (property "Footprint" "" (at 44.45 44.45 0)
-      (effects (font (size 1.27 1.27)) hide)
-    )
-    (property "Datasheet" "" (at 44.45 44.45 0)
-      (effects (font (size 1.27 1.27)) hide)
-    )
-    (pin "1")
-    (instances
-      (project "battery monitoring board"
-        (path "/bf623d80-ca5a-491f-9daa-4dffbeba5279/d1e89632-1041-42ed-815d-03472eda859a"
-          (reference "#PWR029") (unit 1)
         )
       )
@@
         )
         (path "/bf623d80-ca5a-491f-9daa-4dffbeba5279/d1e89632-1041-42ed-815d-03472eda859a"
-          (reference "TP13") (unit 1)
+          (reference "TP1") (unit 1)
         )
       )
@@
   (symbol (lib_id "Device:R_US") (at 62.23 76.2 90) (unit 1)
     (in_bom yes) (on_board yes) (dnp no) (fields_autoplaced)
-    (property "Reference" "R17" (at 62.23 69.85 90)
+    (property "Reference" "R16" (at 62.23 69.85 90)
       (effects (font (size 1.27 1.27)))
     )
@@
       (project "battery monitoring board"
         (path "/bf623d80-ca5a-491f-9daa-4dffbeba5279/d1e89632-1041-42ed-815d-03472eda859a"
-          (reference "R17") (unit 1)
+          (reference "R16") (unit 1)
         )
       )
@@
   (symbol (lib_id "Device:D") (at 72.39 67.31 0) (unit 1)
     (in_bom yes) (on_board yes) (dnp no)
-    (property "Reference" "D7" (at 72.39 62.738 0)
+    (property "Reference" "D6" (at 72.39 62.738 0)
       (effects (font (size 1.27 1.27)))
     )
@@
       (project "battery monitoring board"
         (path "/bf623d80-ca5a-491f-9daa-4dffbeba5279/d1e89632-1041-42ed-815d-03472eda859a"
-          (reference "D7") (unit 1)
+          (reference "D6") (unit 1)
         )
       )
@@
   (symbol (lib_id "Device:R_US") (at 71.12 85.09 0) (unit 1)
     (in_bom yes) (on_board yes) (dnp no) (fields_autoplaced)
-    (property "Reference" "R19" (at 73.66 83.82 0)
+    (property "Reference" "R18" (at 73.66 83.82 0)
       (effects (font (size 1.27 1.27)) (justify left))
     )
@@
       (project "battery monitoring board"
         (path "/bf623d80-ca5a-491f-9daa-4dffbeba5279/d1e89632-1041-42ed-815d-03472eda859a"
-          (reference "R19") (unit 1)
+          (reference "R18") (unit 1)
         )
       )
@@
         )
         (path "/bf623d80-ca5a-491f-9daa-4dffbeba5279/d1e89632-1041-42ed-815d-03472eda859a"
-          (reference "D8") (unit 1)
-        )
-      )
+          (reference "D7") (unit 1)
+        )
+      )
