File: Hardware/battery monitoring board/leak sensor.kicad_sch (KiCad schematic)
At the start: 11 parts, among them J2 Conn_01x02, J3 Conn_01x02, J4 Conn_01x02, J5 Conn_01x02, J6 Conn_01x03, Q1 PNP

Commit message: Revert "Merge branch 'hardware' of https://github.com/bruin-underwater-robotics/2023-2024 into hardware"
This reverts commit 1d5f0f31a35e539c7b0b2eac7ff2db3bf82506a7, reversing
changes made to b9b3862216192341382b87943b4a1d0c2c46b631.
Parts:
- removed D1: D_Photo, symbol Device:D_Photo
- removed J2, J3, J4, J5: Conn_01x02, symbol Connector_Generic:Conn_01x02
- removed J6: Conn_01x03, symbol Connector_Generic:Conn_01x03
- removed Q1: PNP, symbol Simulation_SPICE:PNP
- removed R10: 240, symbol Device:R_US
- removed R7: 27k, symbol Device:R_US
- removed R8, R9: 1k, symbol Device:R_US

Commit message: leak sensor schema
Parts:
- added D1: D_Photo, symbol Device:D_Photo
- added J2, J3, J4, J5: Conn_01x02, symbol Connector_Generic:Conn_01x02
- added J6: Conn_01x03, symbol Connector_Generic:Conn_01x03
- added Q1: PNP, symbol Simulation_SPICE:PNP
- added R10: 240, symbol Device:R_US
- added R7: 27k, symbol Device:R_US
- added R8, R9: 1k, symbol Device:R_US
Connections:
- new net: J2.2 (Pin_2), J3.2 (Pin_2), J4.2 (Pin_2), J5.2 (Pin_2)
- new net: Q1.2 (B), R7.2, R8.2
- new net: D1.2 (A), R10.2
- new net GND: D1.1 (K), J2.1 (Pin_1), J3.1 (Pin_1), J4.1 (Pin_1), J5.1 (Pin_1), J6.1 (Pin_1), R9.2
- new net SIGNAL: J6.3 (Pin_3), Q1.1 (C), R10.1, R9.1
- new net VCC: J6.2 (Pin_2), Q1.3 (E), R7.1
