File: Hardware/battery monitoring board/leak sensor.kicad_sch (KiCad schematic)
At the start: 10 parts, among them J2 Conn_01x02, J3 Conn_01x02, J4 Conn_01x02, J5 Conn_01x02, Q1 PNP

Commit message: changed some minor errors (battery monitoring)
Parts:
- R10: value 100 -> 248
Changed lines of the file:
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@@
       (effects (font (size 1.27 1.27)) (justify left))
     )
-    (property "Value" "100" (at 113.03 71.12 90)
+    (property "Value" "248" (at 113.03 71.12 90)
       (effects (font (size 1.27 1.27)) (justify left))
     )

Commit message: Revert "changed some minor errors (battery monitoring)"
This reverts commit d4ffa11f2369dfdbeb25d57bd1642de1ab50c466.
Parts:
- R10: value 248 -> 100
Changed lines of the file:
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@@
       (effects (font (size 1.27 1.27)) (justify left))
     )
-    (property "Value" "248" (at 113.03 71.12 90)
+    (property "Value" "100" (at 113.03 71.12 90)
       (effects (font (size 1.27 1.27)) (justify left))
     )

Commit message: added programmable LED and reference updates
Parts:
- renumbered D3 to D4
Changed lines of the file:
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@@
   (symbol (lib_id "power:+3V3") (at 105.41 46.99 0) (unit 1)
     (in_bom yes) (on_board yes) (dnp no) (fields_autoplaced)
-    (property "Reference" "#PWR020" (at 105.41 50.8 0)
+    (property "Reference" "#PWR021" (at 105.41 50.8 0)
       (effects (font (size 1.27 1.27)) hide)
     )
@@
       (project "battery monitoring board"
         (path "/bf623d80-ca5a-491f-9daa-4dffbeba5279/7fa71be0-4e2c-431c-85f4-b0f15423b53d"
-          (reference "#PWR020") (unit 1)
+          (reference "#PWR021") (unit 1)
         )
       )
@@
       (project "battery monitoring board"
         (path "/bf623d80-ca5a-491f-9daa-4dffbeba5279/7fa71be0-4e2c-431c-85f4-b0f15423b53d"
-          (reference "#PWR021") (unit 1)
+          (reference "#PWR022") (unit 1)
         )
       )
@@
       (project "battery monitoring board"
         (path "/bf623d80-ca5a-491f-9daa-4dffbeba5279/7fa71be0-4e2c-431c-85f4-b0f15423b53d"
-          (reference "#PWR019") (unit 1)
+          (reference "#PWR020") (unit 1)
         )
       )
@@
       (project "battery monitoring board"
         (path "/bf623d80-ca5a-491f-9daa-4dffbeba5279/7fa71be0-4e2c-431c-85f4-b0f15423b53d"
-          (reference "R11") (unit 1)
+          (reference "R12") (unit 1)
         )
       )
@@
       (project "battery monitoring board"
         (path "/bf623d80-ca5a-491f-9daa-4dffbeba5279/7fa71be0-4e2c-431c-85f4-b0f15423b53d"
-          (reference "R12") (unit 1)
+          (reference "R13") (unit 1)
         )
       )
@@
       (project "battery monitoring board"
         (path "/bf623d80-ca5a-491f-9daa-4dffbeba5279/7fa71be0-4e2c-431c-85f4-b0f15423b53d"
-          (reference "R13") (unit 1)
+          (reference "R14") (unit 1)
         )
       )
@@
   (symbol (lib_id "Device:LED") (at 115.57 80.01 90) (unit 1)
     (in_bom yes) (on_board yes) (dnp no) (fields_autoplaced)
-    (property "Reference" "D3" (at 119.38 80.3275 90)
+    (property "Reference" "D4" (at 119.38 80.3275 90)
       (effects (font (size 1.27 1.27)) (justify right))
     )
@@
       (project "battery monitoring board"
         (path "/bf623d80-ca5a-491f-9daa-4dffbeba5279/7fa71be0-4e2c-431c-85f4-b0f15423b53d"
-          (reference "D3") (unit 1)
+          (reference "D4") (unit 1)
         )
       )
@@
       (project "battery monitoring board"
         (path "/bf623d80-ca5a-491f-9daa-4dffbeba5279/7fa71be0-4e2c-431c-85f4-b0f15423b53d"
-          (reference "R10") (unit 1)
-        )
-      )
+          (reference "R11") (unit 1)
+        )
+      )

Commit message: added test points (battery monitoring)
Parts:
- added TP1: TestPoint, symbol Connector:TestPoint
Connections:
- net LEAK_SIGNAL: now also TP1.1
Changed lines of the file:
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@@
+    )
+  )
+  (symbol (lib_id "Connector:TestPoint") (at 115.57 62.23 0) (unit 1)
+    (in_bom yes) (on_board yes) (dnp no)
+    (property "Reference" "TP1" (at 116.8259 57.15 0)
+      (effects (font (size 1.27 1.27)) (justify left))
+    )
+    (property "Value" "TestPoint" (at 116.8259 58.42 0)
+      (effects (font (size 1.27 1.27)) (justify left))
+    )
+    (property "Footprint" "" (at 120.65 62.23 0)
+      (effects (font (size 1.27 1.27)) hide)
+    )
+    (property "Datasheet" "~" (at 120.65 62.23 0)
+      (effects (font (size 1.27 1.27)) hide)
+    )
+    (pin "1")
+    (instances
+      (project "battery monitoring board"
+        (path "/bf623d80-ca5a-491f-9daa-4dffbeba5279/5ec2dbdf-a276-4d4c-99fc-008475c1e770"
+          (reference "TP1") (unit 1)
+        )
+        (path "/bf623d80-ca5a-491f-9daa-4dffbeba5279/d1e89632-1041-42ed-815d-03472eda859a"
+          (reference "TP9") (unit 1)
+        )
+        (path "/bf623d80-ca5a-491f-9daa-4dffbeba5279/7fa71be0-4e2c-431c-85f4-b0f15423b53d"
+          (reference "TP11") (unit 1)
+        )
+      )
     )
   )

Commit message: Added footprints to battery monitoring
Parts:
- D4: footprint (none) -> Diode_SMD:D_0805_2012Metric_Pad1.15x1.40mm_HandSolder
- J2, J3, J4, J5: footprint (none) -> Library:JST_BM02B-GHS-TBT_LF__SN_
- Q1: footprint (none) -> PCM_4ms_Package_SOT:SOT-23
- R10, R7, R8, R9: footprint (none) -> Resistor_SMD:R_0805_2012Metric_Pad1.20x1.40mm_HandSolder
- TP1: footprint (none) -> Library:Test Pads
Changed lines of the file:
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@@
       (effects (font (size 1.27 1.27)))
     )
-    (property "Footprint" "" (at 36.83 59.69 0)
+    (property "Footprint" "Library:JST_BM02B-GHS-TBT_LF__SN_" (at 36.83 59.69 0)
       (effects (font (size 1.27 1.27)) hide)
     )
@@
       (effects (font (size 1.27 1.27)))
     )
-    (property "Footprint" "" (at 36.83 74.93 0)
+    (property "Footprint" "Library:JST_BM02B-GHS-TBT_LF__SN_" (at 36.83 74.93 0)
       (effects (font (size 1.27 1.27)) hide)
     )
@@
       (effects (font (size 1.27 1.27)) (justify left))
     )
-    (property "Footprint" "" (at 120.65 62.23 0)
+    (property "Footprint" "Library:Test Pads" (at 120.65 62.23 0)
       (effects (font (size 1.27 1.27)) hide)
     )
@@
       (effects (font (size 1.27 1.27)) (justify left))
     )
-    (property "Footprint" "" (at 96.266 52.324 90)
+    (property "Footprint" "Resistor_SMD:R_0805_2012Metric_Pad1.20x1.40mm_HandSolder" (at 96.266 52.324 90)
       (effects (font (size 1.27 1.27)) hide)
     )
@@
       (effects (font (size 1.27 1.27)) (justify left))
     )
-    (property "Footprint" "" (at 106.426 70.104 90)
+    (property "Footprint" "Resistor_SMD:R_0805_2012Metric_Pad1.20x1.40mm_HandSolder" (at 106.426 70.104 90)
       (effects (font (size 1.27 1.27)) hide)
     )
@@
       (effects (font (size 1.27 1.27)) (justify left))
     )
-    (property "Footprint" "" (at 116.586 70.104 90)
+    (property "Footprint" "Resistor_SMD:R_0805_2012Metric_Pad1.20x1.40mm_HandSolder" (at 116.586 70.104 90)
       (effects (font (size 1.27 1.27)) hide)
     )
@@
       (effects (font (size 1.27 1.27)))
     )
-    (property "Footprint" "" (at 36.83 67.31 0)
+    (property "Footprint" "Library:JST_BM02B-GHS-TBT_LF__SN_" (at 36.83 67.31 0)
       (effects (font (size 1.27 1.27)) hide)
     )
@@
       (effects (font (size 1.27 1.27)))
     )
-    (property "Footprint" "" (at 36.83 52.07 0)
+    (property "Footprint" "Library:JST_BM02B-GHS-TBT_LF__SN_" (at 36.83 52.07 0)
       (effects (font (size 1.27 1.27)) hide)
     )
@@
       (effects (font (size 1.27 1.27)) (justify right))
     )
-    (property "Footprint" "" (at 115.57 80.01 0)
+    (property "Footprint" "Diode_SMD:D_0805_2012Metric_Pad1.15x1.40mm_HandSolder" (at 115.57 80.01 0)
       (effects (font (size 1.27 1.27)) hide)
     )
@@
       (effects (font (size 1.27 1.27)))
     )
-    (property "Footprint" "" (at 86.614 54.864 90)
+    (property "Footprint" "Resistor_SMD:R_0805_2012Metric_Pad1.20x1.40mm_HandSolder" (at 86.614 54.864 90)
       (effects (font (size 1.27 1.27)) hide)
     )
@@
       (effects (font (size 1.27 1.27)) (justify left))
     )
-    (property "Footprint" "" (at 138.43 55.88 0)
-      (effects (font (size 1.27 1.27)) hide)
-    )
+    (property "Footprint" "PCM_4ms_Package_SOT:SOT-23" (at 138.43 55.88 0)
+      (effects (font (size 1.27 1.27)) hide)
+    )

Commit message: Update leak sensor.kicad_sch
Connections:
- net +3V3: now also Q1.2 (E); no longer Q1.3 (E)
- net LEAK_SIGNAL: now also Q1.3 (C); no longer Q1.1 (C)
- net at R7.2, R8.2: now also Q1.1 (B); no longer Q1.2 (B)
Changed lines of the file:
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@@
       (effects (font (size 1.27 1.27)) hide)
     )
-    (property "Sim.Device" "PNP" (at 102.87 55.88 0)
+    (property "Sim.Device" "PNP" (at 91.44 53.34 0)
       (effects (font (size 1.27 1.27)) hide)
     )
-    (property "Sim.Type" "GUMMELPOON" (at 102.87 55.88 0)
+    (property "Sim.Type" "GUMMELPOON" (at 95.25 50.8 0)
       (effects (font (size 1.27 1.27)) hide)
     )
-    (property "Sim.Pins" "1=C 2=B 3=E" (at 102.87 55.88 0)
+    (property "Sim.Pins" "1=B 2=E 3=C" (at 95.25 48.26 0)
       (effects (font (size 1.27 1.27)) hide)
     )
+    (pin "3")
     (pin "1")
     (pin "2")
-    (pin "3")
     (instances
       (project "leak sensor"
