File: Hardware/battery monitoring board/battery monitoring board.kicad_sch (KiCad schematic)
At the start: 1 part

Commit message: Added power connectors
Parts:
- added J7, J8: Conn_01x02, symbol Connector_Generic:Conn_01x02
Connections:
- net GND: now also J7.1 (Pin_1), J8.2 (Pin_2)
- new net e-switch/BATTERY_IN: J7.2 (Pin_2)
- new net e-switch/SYSTEM_POWER: J8.1 (Pin_1)
Other:
- sheet e-switch ports: added BATTERY_IN, SYSTEM_POWER; removed none
Changed lines of the file:
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@@
+    (stroke (width 0) (type default))
+  )
+  (wire (pts (xy 184.15 71.12) (xy 191.77 71.12))
     (stroke (width 0) (type default))
   )
@@
   )
   (wire (pts (xy 148.59 101.6) (xy 153.67 101.6))
+    (stroke (width 0) (type default))
+  )
+  (wire (pts (xy 147.32 71.12) (xy 153.67 71.12))
     (stroke (width 0) (type default))
   )
@@
     )
   )
+  (symbol (lib_id "Connector_Generic:Conn_01x02") (at 196.85 71.12 0) (unit 1)
+    (in_bom yes) (on_board yes) (dnp no) (fields_autoplaced)
+    (property "Reference" "J8" (at 199.39 71.12 0)
+      (effects (font (size 1.27 1.27)) (justify left))
+    )
+    (property "Value" "Conn_01x02" (at 199.39 73.66 0)
+      (effects (font (size 1.27 1.27)) (justify left))
+    )
+    (property "Footprint" "" (at 196.85 71.12 0)
+      (effects (font (size 1.27 1.27)) hide)
+    )
+    (property "Datasheet" "~" (at 196.85 71.12 0)
+      (effects (font (size 1.27 1.27)) hide)
+    )
+    (pin "1")
+    (pin "2")
+    (instances
+      (project "battery monitoring board"
+        (path "/bf623d80-ca5a-491f-9daa-4dffbeba5279"
+          (reference "J8") (unit 1)
+        )
+      )
+    )
+  )
   (symbol (lib_id "power:+3V3") (at 124.46 58.42 0) (unit 1)
     (in_bom yes) (on_board yes) (dnp no)
@@
     )
   )
+  (symbol (lib_id "PCM_4ms_Power-symbol:GND") (at 191.77 73.66 0) (unit 1)
+    (in_bom yes) (on_board yes) (dnp no)
+    (property "Reference" "#PWR020" (at 191.77 80.01 0)
+      (effects (font (size 1.27 1.27)) hide)
+    )
+    (property "Value" "GND" (at 194.31 76.2 0)
+      (effects (font (size 1.27 1.27)))
+    )
+    (property "Footprint" "" (at 191.77 73.66 0)
+      (effects (font (size 1.27 1.27)) hide)
+    )
+    (property "Datasheet" "" (at 191.77 73.66 0)
+      (effects (font (size 1.27 1.27)) hide)
+    )
+    (pin "1")
+    (instances
+      (project "battery monitoring board"
+        (path "/bf623d80-ca5a-491f-9daa-4dffbeba5279"
+          (reference "#PWR020") (unit 1)
+        )
+      )
+    )
+  )
   (symbol (lib_id "PCM_4ms_Power-symbol:GND") (at 121.92 113.03 0) (unit 1)
     (in_bom yes) (on_board yes) (dnp no) (fields_autoplaced)
@@
     )
   )
+  (symbol (lib_id "Connector_Generic:Conn_01x02") (at 142.24 73.66 180) (unit 1)
+    (in_bom yes) (on_board yes) (dnp no) (fields_autoplaced)
+    (property "Reference" "J7" (at 142.24 64.77 0)
+      (effects (font (size 1.27 1.27)))
+    )
+    (property "Value" "Conn_01x02" (at 142.24 67.31 0)
+      (effects (font (size 1.27 1.27)))
+    )
+    (property "Footprint" "" (at 142.24 73.66 0)
+      (effects (font (size 1.27 1.27)) hide)
+    )
+    (property "Datasheet" "~" (at 142.24 73.66 0)
+      (effects (font (size 1.27 1.27)) hide)
+    )
+    (pin "1")
+    (pin "2")
+    (instances
+      (project "battery monitoring board"
+        (path "/bf623d80-ca5a-491f-9daa-4dffbeba5279"
+          (reference "J7") (unit 1)
+        )
+      )
+    )
+  )
   (symbol (lib_id "PCM_4ms_Power-symbol:+5V") (at 127 58.42 0) (unit 1)
     (in_bom yes) (on_board yes) (dnp no)
@@
         (path "/bf623d80-ca5a-491f-9daa-4dffbeba5279"
           (reference "#PWR02") (unit 1)
+        )
+      )
+    )
+  )
+  (symbol (lib_id "PCM_4ms_Power-symbol:GND") (at 147.32 73.66 0) (unit 1)
+    (in_bom yes) (on_board yes) (dnp no)
+    (property "Reference" "#PWR021" (at 147.32 80.01 0)
+      (effects (font (size 1.27 1.27)) hide)
+    )
+    (property "Value" "GND" (at 149.86 76.2 0)
+      (effects (font (size 1.27 1.27)))
+    )
+    (property "Footprint" "" (at 147.32 73.66 0)
+      (effects (font (size 1.27 1.27)) hide)
+    )
+    (property "Datasheet" "" (at 147.32 73.66 0)
+      (effects (font (size 1.27 1.27)) hide)
+    )
+    (pin "1")
+    (instances
+      (project "battery monitoring board"
+        (path "/bf623d80-ca5a-491f-9daa-4dffbeba5279"
+          (reference "#PWR021") (unit 1)
         )
       )
@@
       (effects (font (size 1.27 1.27)) (justify right))
     )
-    (pin "so" input (at 85.09 100.33 0)
+    (pin "so" output (at 85.09 100.33 0)
       (effects (font (size 1.27 1.27)) (justify right))
     )
@@
       (effects (font (size 1.27 1.27)) (justify left top))
     )
-    (pin "LEAK_SIGNAL" input (at 85.09 74.93 0)
+    (pin "LEAK_SIGNAL" output (at 85.09 74.93 0)
       (effects (font (size 1.27 1.27)) (justify right))
     )
@@
     )
   )
-  (sheet (at 153.67 66.802) (size 30.48 19.304) (fields_autoplaced)
+  (sheet (at 153.67 66.802) (size 30.48 19.304)
     (stroke (width 0.1524) (type solid))
     (fill (color 0 0 0 0.0000))
@@
       (effects (font (size 1.27 1.27)) (justify left))
     )
+    (pin "SYSTEM_POWER" output (at 184.15 71.12 0)
+      (effects (font (size 1.27 1.27)) (justify right))
+    )
+    (pin "BATTERY_IN" input (at 153.67 71.12 180)
+      (effects (font (size 1.27 1.27)) (justify left))
+    )

Commit message: Updated reference labels
Parts:
- renumbered J7 to J1, J8 to J2
Changed lines of the file:
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@@
   (symbol (lib_id "Connector_Generic:Conn_01x02") (at 196.85 71.12 0) (unit 1)
     (in_bom yes) (on_board yes) (dnp no) (fields_autoplaced)
-    (property "Reference" "J8" (at 199.39 71.12 0)
+    (property "Reference" "J2" (at 199.39 71.12 0)
       (effects (font (size 1.27 1.27)) (justify left))
     )
@@
       (project "battery monitoring board"
         (path "/bf623d80-ca5a-491f-9daa-4dffbeba5279"
-          (reference "J8") (unit 1)
+          (reference "J2") (unit 1)
         )
       )
@@
   (symbol (lib_id "power:+3V3") (at 124.46 58.42 0) (unit 1)
     (in_bom yes) (on_board yes) (dnp no)
-    (property "Reference" "#PWR019" (at 124.46 62.23 0)
+    (property "Reference" "#PWR02" (at 124.46 62.23 0)
       (effects (font (size 1.27 1.27)) hide)
     )
@@
       (project "battery monitoring board"
         (path "/bf623d80-ca5a-491f-9daa-4dffbeba5279"
-          (reference "#PWR019") (unit 1)
+          (reference "#PWR02") (unit 1)
         )
       )
@@
   (symbol (lib_id "PCM_4ms_Power-symbol:GND") (at 191.77 73.66 0) (unit 1)
     (in_bom yes) (on_board yes) (dnp no)
-    (property "Reference" "#PWR020" (at 191.77 80.01 0)
+    (property "Reference" "#PWR05" (at 191.77 80.01 0)
       (effects (font (size 1.27 1.27)) hide)
     )
@@
       (project "battery monitoring board"
         (path "/bf623d80-ca5a-491f-9daa-4dffbeba5279"
-          (reference "#PWR020") (unit 1)
+          (reference "#PWR05") (unit 1)
         )
       )
@@
   (symbol (lib_id "Connector_Generic:Conn_01x02") (at 142.24 73.66 180) (unit 1)
     (in_bom yes) (on_board yes) (dnp no) (fields_autoplaced)
-    (property "Reference" "J7" (at 142.24 64.77 0)
+    (property "Reference" "J1" (at 142.24 64.77 0)
       (effects (font (size 1.27 1.27)))
     )
@@
       (project "battery monitoring board"
         (path "/bf623d80-ca5a-491f-9daa-4dffbeba5279"
-          (reference "J7") (unit 1)
+          (reference "J1") (unit 1)
         )
       )
@@
   (symbol (lib_id "PCM_4ms_Power-symbol:+5V") (at 127 58.42 0) (unit 1)
     (in_bom yes) (on_board yes) (dnp no)
-    (property "Reference" "#PWR02" (at 127 62.23 0)
+    (property "Reference" "#PWR03" (at 127 62.23 0)
       (effects (font (size 1.27 1.27)) hide)
     )
@@
       (project "battery monitoring board"
         (path "/bf623d80-ca5a-491f-9daa-4dffbeba5279"
-          (reference "#PWR02") (unit 1)
+          (reference "#PWR03") (unit 1)
         )
       )
@@
   (symbol (lib_id "PCM_4ms_Power-symbol:GND") (at 147.32 73.66 0) (unit 1)
     (in_bom yes) (on_board yes) (dnp no)
-    (property "Reference" "#PWR021" (at 147.32 80.01 0)
+    (property "Reference" "#PWR04" (at 147.32 80.01 0)
       (effects (font (size 1.27 1.27)) hide)
     )
@@
       (project "battery monitoring board"
         (path "/bf623d80-ca5a-491f-9daa-4dffbeba5279"
-          (reference "#PWR021") (unit 1)
+          (reference "#PWR04") (unit 1)
         )
       )

Commit message: Revert "Updated reference labels"
This reverts commit 7ccd23260c988ead49c0bcfa936e50f6d09a7000.
Parts:
- renumbered J1 to J7, J2 to J8
Changed lines of the file:
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@@
   (symbol (lib_id "Connector_Generic:Conn_01x02") (at 196.85 71.12 0) (unit 1)
     (in_bom yes) (on_board yes) (dnp no) (fields_autoplaced)
-    (property "Reference" "J2" (at 199.39 71.12 0)
+    (property "Reference" "J8" (at 199.39 71.12 0)
       (effects (font (size 1.27 1.27)) (justify left))
     )
@@
       (project "battery monitoring board"
         (path "/bf623d80-ca5a-491f-9daa-4dffbeba5279"
-          (reference "J2") (unit 1)
+          (reference "J8") (unit 1)
         )
       )
@@
   (symbol (lib_id "power:+3V3") (at 124.46 58.42 0) (unit 1)
     (in_bom yes) (on_board yes) (dnp no)
-    (property "Reference" "#PWR02" (at 124.46 62.23 0)
+    (property "Reference" "#PWR019" (at 124.46 62.23 0)
       (effects (font (size 1.27 1.27)) hide)
     )
@@
       (project "battery monitoring board"
         (path "/bf623d80-ca5a-491f-9daa-4dffbeba5279"
-          (reference "#PWR02") (unit 1)
+          (reference "#PWR019") (unit 1)
         )
       )
@@
   (symbol (lib_id "PCM_4ms_Power-symbol:GND") (at 191.77 73.66 0) (unit 1)
     (in_bom yes) (on_board yes) (dnp no)
-    (property "Reference" "#PWR05" (at 191.77 80.01 0)
+    (property "Reference" "#PWR020" (at 191.77 80.01 0)
       (effects (font (size 1.27 1.27)) hide)
     )
@@
       (project "battery monitoring board"
         (path "/bf623d80-ca5a-491f-9daa-4dffbeba5279"
-          (reference "#PWR05") (unit 1)
+          (reference "#PWR020") (unit 1)
         )
       )
@@
   (symbol (lib_id "Connector_Generic:Conn_01x02") (at 142.24 73.66 180) (unit 1)
     (in_bom yes) (on_board yes) (dnp no) (fields_autoplaced)
-    (property "Reference" "J1" (at 142.24 64.77 0)
+    (property "Reference" "J7" (at 142.24 64.77 0)
       (effects (font (size 1.27 1.27)))
     )
@@
       (project "battery monitoring board"
         (path "/bf623d80-ca5a-491f-9daa-4dffbeba5279"
-          (reference "J1") (unit 1)
+          (reference "J7") (unit 1)
         )
       )
@@
   (symbol (lib_id "PCM_4ms_Power-symbol:+5V") (at 127 58.42 0) (unit 1)
     (in_bom yes) (on_board yes) (dnp no)
-    (property "Reference" "#PWR03" (at 127 62.23 0)
+    (property "Reference" "#PWR02" (at 127 62.23 0)
       (effects (font (size 1.27 1.27)) hide)
     )
@@
       (project "battery monitoring board"
         (path "/bf623d80-ca5a-491f-9daa-4dffbeba5279"
-          (reference "#PWR03") (unit 1)
+          (reference "#PWR02") (unit 1)
         )
       )
@@
   (symbol (lib_id "PCM_4ms_Power-symbol:GND") (at 147.32 73.66 0) (unit 1)
     (in_bom yes) (on_board yes) (dnp no)
-    (property "Reference" "#PWR04" (at 147.32 80.01 0)
+    (property "Reference" "#PWR021" (at 147.32 80.01 0)
       (effects (font (size 1.27 1.27)) hide)
     )
@@
       (project "battery monitoring board"
         (path "/bf623d80-ca5a-491f-9daa-4dffbeba5279"
-          (reference "#PWR04") (unit 1)
+          (reference "#PWR021") (unit 1)
         )
       )
